File: kiCad/keyboard.kicad_pcb (KiCad board)
At the start: 2 copper layers, 123 parts, among them J0 Conn_01x03, SW1 MX, SW10 MX, SW11 MX, SW12 MX, SW13 MX, SW14 MX, SW15 MX, SW16 MX, SW17 MX, SW18 MX, SW19 MX, SW2 MX, SW20 MX, SW21 MX, SW22 MX, SW23 MX, SW24 MX, SW25 MX, SW26 MX, SW27 MX, SW28 MX, SW29 MX, SW3 MX, SW30 MX, SW31 MX, SW32 MX, SW33 MX, SW34 MX, SW35 MX, SW36 MX, SW37 MX, SW38 MX, SW39 MX, SW4 MX, SW40 MX, SW41 MX, SW42 MX, SW43 MX, SW44 MX, SW45 MX, SW46 MX, SW47 MX, SW48 MX, SW49 MX, SW5 MX, SW50 MX, SW51 MX, SW52 MX, SW53 MX, SW54 MX, SW55 MX, SW56 MX, SW57 MX, SW58 MX, SW59 MX, SW6 MX, SW60 MX, SW61 MX, SW7 MX, SW8 MX, SW9 MX, U0 Sparkfun_Pro_Micro

Commit message: draw pcb, add more footprints
Parts:
- removed D60: D, Diode_THT:D_DO-35_SOD27_P7.62mm_Horizontal
- removed SW60: MX, Button_Switch_Keyboard:SW_Cherry_MX_1.00u_PCB
- added D0: 1N4148, Diode_THT:D_DO-35_SOD27_P7.62mm_Horizontal, F.Cu at (52.4, 55.4)
- added SW0: MX, MX_Alps_Hybrid:MX-1U-NoLED, F.Cu at (42.9, 52.4)
- D1, D10, D11, D12, D13, D14, D15, D16, D17, D18, D19, D2, D20, D21, D22, D23, D24, D25, D26, D27, D28, D29, D3, D30, D31, D32, D33, D34, D35, D36, D37, D38, D39, D4, D40, D41, D42, D43, D44, D45, D46, D47, D48, D49, D5, D50, D51, D52, D53, D54, D55, D56, D57, D58, D59, D6, D7, D8, D9: value D -> 1N4148
- SW1, SW10, SW11, SW12, SW13, SW14, SW15, SW16, SW17, SW18, SW19, SW2, SW20, SW21, SW22, SW23, SW24, SW25, SW26, SW27, SW28, SW29, SW3, SW30, SW31, SW32, SW33, SW34, SW35, SW36, SW37, SW38, SW39, SW4, SW40, SW41, SW42, SW43, SW44, SW45, SW46, SW47, SW48, SW49, SW5, SW50, SW51, SW52, SW53, SW54, SW55, SW56, SW57, SW58, SW59, SW6, SW7, SW8, SW9: footprint Button_Switch_Keyboard:SW_Cherry_MX_1.00u_PCB -> MX_Alps_Hybrid:MX-1U-NoLED
- SW61: footprint Button_Switch_Keyboard:SW_Cherry_MX_1.00u_PCB -> Molex-0548190589:PushButton_6x6mm_TH_Pretty; moved to B.Cu
- U0: moved to B.Cu
- moved J0 238.0 mm to (46.2, 42.9), turned to -90 degrees
- moved D46 215.0 mm to (236.4, 100.0), turned to 180 degrees
- moved D24 214.2 mm to (52.4, 75.2), turned to 90 degrees
- moved D2 204.5 mm to (57.1, 42.9)
- moved D13 201.0 mm to (62.7, 61.9)
- moved D45 195.5 mm to (223.8, 94.3), turned to 90 degrees
- moved D25 193.4 mm to (71.4, 75.2), turned to 90 degrees
- moved D47 183.8 mm to (242.9, 93.5), turned to 90 degrees
- moved D19 181.4 mm to (185.7, 55.4), turned to 90 degrees
- moved SW20 179.2 mm to (195.3, 52.4)
- moved D22 178.1 mm to (242.9, 55.4), turned to 90 degrees
- moved D35 175.3 mm to (247.8, 81.0)
- moved D33 174.4 mm to (223.8, 75.2), turned to 90 degrees
- moved D12 172.4 mm to (247.7, 42.9)
- moved D14 168.3 mm to (94.3, 61.9), turned to 180 degrees
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Connections:
- D1 pad 1: Net-(D1-Pad1) -> /ROW0
- D1 pad 2: /COL0 -> Net-(D1-Pad2)
- D10 pad 1: Net-(D10-Pad1) -> /ROW0
- D10 pad 2: /COL9 -> Net-(SW10-Pad2)
- D11 pad 1: Net-(D11-Pad1) -> /ROW0
- D11 pad 2: /COL10 -> Net-(SW11-Pad2)
- D12 pad 1: Net-(D12-Pad1) -> /ROW0
- D12 pad 2: /COL11 -> Net-(SW12-Pad2)
- D13 pad 1: Net-(D13-Pad1) -> /ROW1
- D13 pad 2: /COL0 -> Net-(D13-Pad2)
- D14 pad 1: Net-(D14-Pad1) -> /ROW1
- D14 pad 2: /COL1 -> Net-(D14-Pad2)
- D15 pad 1: Net-(D15-Pad1) -> /ROW1
- D15 pad 2: /COL2 -> Net-(D15-Pad2)
- D16 pad 1: Net-(D16-Pad1) -> /ROW1
- D16 pad 2: /COL3 -> Net-(D16-Pad2)
- D17 pad 1: Net-(D17-Pad1) -> /ROW1
- D17 pad 2: /COL4 -> Net-(D17-Pad2)
- D18 pad 1: Net-(D18-Pad1) -> /ROW1
- D18 pad 2: /COL5 -> Net-(D18-Pad2)
- D19 pad 1: Net-(D19-Pad1) -> /ROW1
- D19 pad 2: /COL6 -> Net-(D19-Pad2)
- D2 pad 1: Net-(D2-Pad1) -> /ROW0
- D2 pad 2: /COL1 -> Net-(SW2-Pad2)
- D20 pad 1: Net-(D20-Pad1) -> /ROW1
- D20 pad 2: /COL7 -> Net-(D20-Pad2)
- D21 pad 1: Net-(D21-Pad1) -> /ROW1
- D21 pad 2: /COL8 -> Net-(D21-Pad2)
- D22 pad 1: Net-(D22-Pad1) -> /ROW1
- D22 pad 2: /COL9 -> Net-(D22-Pad2)
- D23 pad 1: Net-(D23-Pad1) -> /ROW1
- D23 pad 2: /COL10 -> Net-(D23-Pad2)
- D24 pad 1: Net-(D24-Pad1) -> /ROW2
- D24 pad 2: /COL11 -> Net-(D24-Pad2)
- D25 pad 1: Net-(D25-Pad1) -> /ROW2
- D25 pad 2: /COL0 -> Net-(D25-Pad2)
- D26 pad 1: Net-(D26-Pad1) -> /ROW2
- D26 pad 2: /COL1 -> Net-(D26-Pad2)
- D27 pad 1: Net-(D27-Pad1) -> /ROW2
- D27 pad 2: /COL2 -> Net-(D27-Pad2)
- D28 pad 1: Net-(D28-Pad1) -> /ROW2
- D28 pad 2: /COL3 -> Net-(D28-Pad2)
- D29 pad 1: Net-(D29-Pad1) -> /ROW2
- D29 pad 2: /COL4 -> Net-(D29-Pad2)
- D3 pad 1: Net-(D3-Pad1) -> /ROW0
- D3 pad 2: /COL2 -> Net-(SW3-Pad2)
- D30 pad 1: Net-(D30-Pad1) -> /ROW2
- D30 pad 2: /COL5 -> Net-(D30-Pad2)
- D31 pad 1: Net-(D31-Pad1) -> /ROW2
- D31 pad 2: /COL6 -> Net-(D31-Pad2)
- D32 pad 1: Net-(D32-Pad1) -> /ROW2
- D32 pad 2: /COL7 -> Net-(D32-Pad2)
- D33 pad 1: Net-(D33-Pad1) -> /ROW2
- D33 pad 2: /COL8 -> Net-(D33-Pad2)
- D34 pad 1: Net-(D34-Pad1) -> /ROW2
- D34 pad 2: /COL9 -> Net-(D34-Pad2)
- D35 pad 1: Net-(D35-Pad1) -> /ROW2
- D35 pad 2: /COL10 -> Net-(D35-Pad2)
- D36 pad 1: Net-(D36-Pad1) -> /ROW3
- D36 pad 2: /COL11 -> Net-(D36-Pad2)
- D37 pad 1: Net-(D37-Pad1) -> /ROW3
- D37 pad 2: /COL0 -> Net-(D37-Pad2)
- D38 pad 1: Net-(D38-Pad1) -> /ROW3
- D38 pad 2: /COL1 -> Net-(D38-Pad2)
- D39 pad 1: Net-(D39-Pad1) -> /ROW3
- D39 pad 2: /COL2 -> Net-(D39-Pad2)
- D4 pad 1: Net-(D4-Pad1) -> /ROW0
- D4 pad 2: /COL3 -> Net-(SW4-Pad2)
- D40 pad 1: Net-(D40-Pad1) -> /ROW3
- D40 pad 2: /COL3 -> Net-(D40-Pad2)
- D41 pad 1: Net-(D41-Pad1) -> /ROW3
- D41 pad 2: /COL4 -> Net-(D41-Pad2)
- D42 pad 1: Net-(D42-Pad1) -> /ROW3
- D42 pad 2: /COL5 -> Net-(D42-Pad2)
- D43 pad 1: Net-(D43-Pad1) -> /ROW3
- D43 pad 2: /COL6 -> Net-(D43-Pad2)
- D44 pad 1: Net-(D44-Pad1) -> /ROW3
- D44 pad 2: /COL7 -> Net-(D44-Pad2)
- D45 pad 1: Net-(D45-Pad1) -> /ROW3
- D45 pad 2: /COL8 -> Net-(D45-Pad2)
- D46 pad 1: Net-(D46-Pad1) -> /ROW3
- D46 pad 2: /COL9 -> Net-(D46-Pad2)
- D47 pad 1: Net-(D47-Pad1) -> /ROW3
- D47 pad 2: /COL10 -> Net-(D47-Pad2)
- D48 pad 1: Net-(D48-Pad1) -> /ROW4
- D48 pad 2: /COL11 -> Net-(D48-Pad2)
- D49 pad 1: Net-(D49-Pad1) -> /ROW4
- D49 pad 2: /COL0 -> Net-(D49-Pad2)
- D5 pad 1: Net-(D5-Pad1) -> /ROW0
- D5 pad 2: /COL4 -> Net-(SW5-Pad2)
- D50 pad 1: Net-(D50-Pad1) -> /ROW4
- D50 pad 2: /COL1 -> Net-(D50-Pad2)
- D51 pad 1: Net-(D51-Pad1) -> /ROW4
- D51 pad 2: /COL2 -> Net-(D51-Pad2)
- D52 pad 1: Net-(D52-Pad1) -> /ROW4
- D52 pad 2: /COL3 -> Net-(D52-Pad2)
- D53 pad 1: Net-(D53-Pad1) -> /ROW4
- D53 pad 2: /COL4 -> Net-(D53-Pad2)
- D54 pad 1: Net-(D54-Pad1) -> /ROW4
- D54 pad 2: /COL5 -> Net-(D54-Pad2)
- D55 pad 1: Net-(D55-Pad1) -> /ROW4
- D55 pad 2: /COL6 -> Net-(D55-Pad2)
- D56 pad 1: Net-(D56-Pad1) -> /ROW4
- D56 pad 2: /COL7 -> Net-(D56-Pad2)
- D57 pad 1: Net-(D57-Pad1) -> /ROW4
- D57 pad 2: /COL8 -> Net-(D57-Pad2)
- D58 pad 1: Net-(D58-Pad1) -> /ROW4
- D58 pad 2: /COL9 -> Net-(D58-Pad2)
- D59 pad 1: Net-(D59-Pad1) -> /ROW4
- D59 pad 2: /COL10 -> Net-(D59-Pad2)
- D6 pad 1: Net-(D6-Pad1) -> /ROW0
- D6 pad 2: /COL5 -> Net-(SW6-Pad2)
- D7 pad 1: Net-(D7-Pad1) -> /ROW0
- D7 pad 2: /COL6 -> Net-(D7-Pad2)
- D8 pad 1: Net-(D8-Pad1) -> /ROW0
- D8 pad 2: /COL7 -> Net-(SW8-Pad2)
- D9 pad 1: Net-(D9-Pad1) -> /ROW0
- D9 pad 2: /COL8 -> Net-(SW9-Pad2)
- SW1 pad 1: /ROW0 -> /COL0
- SW1 pad 2: Net-(D1-Pad1) -> Net-(D1-Pad2)
- SW10 pad 1: /ROW0 -> /COL9
- SW10 pad 2: Net-(D10-Pad1) -> Net-(SW10-Pad2)
- SW11 pad 1: /ROW0 -> /COL10
- SW11 pad 2: Net-(D11-Pad1) -> Net-(SW11-Pad2)
- SW12 pad 1: /ROW0 -> /COL11
- SW12 pad 2: Net-(D12-Pad1) -> Net-(SW12-Pad2)
- SW13 pad 1: /ROW1 -> /COL1
- SW13 pad 2: Net-(D13-Pad1) -> Net-(D13-Pad2)
- SW14 pad 1: /ROW1 -> /COL2
- SW14 pad 2: Net-(D14-Pad1) -> Net-(D14-Pad2)
- SW15 pad 1: /ROW1 -> /COL3
- SW15 pad 2: Net-(D15-Pad1) -> Net-(D15-Pad2)
- SW16 pad 1: /ROW1 -> /COL4
- SW16 pad 2: Net-(D16-Pad1) -> Net-(D16-Pad2)
- SW17 pad 1: /ROW1 -> /COL5
- SW17 pad 2: Net-(D17-Pad1) -> Net-(D17-Pad2)
- SW18 pad 1: /ROW1 -> /COL6
- SW18 pad 2: Net-(D18-Pad1) -> Net-(D18-Pad2)
- SW19 pad 1: /ROW1 -> /COL7
- SW19 pad 2: Net-(D19-Pad1) -> Net-(D19-Pad2)
- SW2 pad 1: /ROW0 -> /COL1
- SW2 pad 2: Net-(D2-Pad1) -> Net-(SW2-Pad2)
- SW20 pad 1: /ROW1 -> /COL8
- SW20 pad 2: Net-(D20-Pad1) -> Net-(D20-Pad2)
- SW21 pad 1: /ROW1 -> /COL9
- SW21 pad 2: Net-(D21-Pad1) -> Net-(D21-Pad2)
- SW22 pad 1: /ROW1 -> /COL10
- SW22 pad 2: Net-(D22-Pad1) -> Net-(D22-Pad2)
- SW23 pad 1: /ROW1 -> /COL11
- SW23 pad 2: Net-(D23-Pad1) -> Net-(D23-Pad2)
- SW24 pad 1: /ROW1 -> /COL0
- SW24 pad 2: Net-(D24-Pad1) -> Net-(D24-Pad2)
- SW25 pad 1: /ROW2 -> /COL1
- SW25 pad 2: Net-(D25-Pad1) -> Net-(D25-Pad2)
- SW26 pad 1: /ROW2 -> /COL2
- SW26 pad 2: Net-(D26-Pad1) -> Net-(D26-Pad2)
- SW27 pad 1: /ROW2 -> /COL3
- SW27 pad 2: Net-(D27-Pad1) -> Net-(D27-Pad2)
- SW28 pad 1: /ROW2 -> /COL4
- SW28 pad 2: Net-(D28-Pad1) -> Net-(D28-Pad2)
- SW29 pad 1: /ROW2 -> /COL5
- SW29 pad 2: Net-(D29-Pad1) -> Net-(D29-Pad2)
- SW3 pad 1: /ROW0 -> /COL2
- SW3 pad 2: Net-(D3-Pad1) -> Net-(SW3-Pad2)
- SW30 pad 1: /ROW2 -> /COL6
- SW30 pad 2: Net-(D30-Pad1) -> Net-(D30-Pad2)
- SW31 pad 1: /ROW2 -> /COL7
- SW31 pad 2: Net-(D31-Pad1) -> Net-(D31-Pad2)
- SW32 pad 1: /ROW2 -> /COL8
- SW32 pad 2: Net-(D32-Pad1) -> Net-(D32-Pad2)
- SW33 pad 1: /ROW2 -> /COL9
- SW33 pad 2: Net-(D33-Pad1) -> Net-(D33-Pad2)
- SW34 pad 1: /ROW2 -> /COL10
- SW34 pad 2: Net-(D34-Pad1) -> Net-(D34-Pad2)
- SW35 pad 1: /ROW2 -> /COL11
- SW35 pad 2: Net-(D35-Pad1) -> Net-(D35-Pad2)
- SW36 pad 1: /ROW2 -> /COL0
- SW36 pad 2: Net-(D36-Pad1) -> Net-(D36-Pad2)
- SW37 pad 1: /ROW3 -> /COL1
- SW37 pad 2: Net-(D37-Pad1) -> Net-(D37-Pad2)
- SW38 pad 1: /ROW3 -> /COL2
- SW38 pad 2: Net-(D38-Pad1) -> Net-(D38-Pad2)
- SW39 pad 1: /ROW3 -> /COL3
- SW39 pad 2: Net-(D39-Pad1) -> Net-(D39-Pad2)
- SW4 pad 1: /ROW0 -> /COL3
- SW4 pad 2: Net-(D4-Pad1) -> Net-(SW4-Pad2)
- SW40 pad 1: /ROW3 -> /COL4
- SW40 pad 2: Net-(D40-Pad1) -> Net-(D40-Pad2)
- SW41 pad 1: /ROW3 -> /COL5
- SW41 pad 2: Net-(D41-Pad1) -> Net-(D41-Pad2)
- SW42 pad 1: /ROW3 -> /COL6
- SW42 pad 2: Net-(D42-Pad1) -> Net-(D42-Pad2)
- SW43 pad 1: /ROW3 -> /COL7
- SW43 pad 2: Net-(D43-Pad1) -> Net-(D43-Pad2)
- SW44 pad 1: /ROW3 -> /COL8
- SW44 pad 2: Net-(D44-Pad1) -> Net-(D44-Pad2)
- SW45 pad 1: /ROW3 -> /COL9
- SW45 pad 2: Net-(D45-Pad1) -> Net-(D45-Pad2)
- SW46 pad 1: /ROW3 -> /COL10
- SW46 pad 2: Net-(D46-Pad1) -> Net-(D46-Pad2)
- SW47 pad 1: /ROW3 -> /COL11
- SW47 pad 2: Net-(D47-Pad1) -> Net-(D47-Pad2)
- SW48 pad 1: /ROW3 -> /COL0
- SW48 pad 2: Net-(D48-Pad1) -> Net-(D48-Pad2)
- SW49 pad 1: /ROW4 -> /COL1
- SW49 pad 2: Net-(D49-Pad1) -> Net-(D49-Pad2)
- SW5 pad 1: /ROW0 -> /COL4
- SW5 pad 2: Net-(D5-Pad1) -> Net-(SW5-Pad2)
- SW50 pad 1: /ROW4 -> /COL2
- SW50 pad 2: Net-(D50-Pad1) -> Net-(D50-Pad2)
- SW51 pad 1: /ROW4 -> /COL3
- SW51 pad 2: Net-(D51-Pad1) -> Net-(D51-Pad2)
- SW52 pad 1: /ROW4 -> /COL4
- SW52 pad 2: Net-(D52-Pad1) -> Net-(D52-Pad2)
- SW53 pad 1: /ROW4 -> /COL5
- SW53 pad 2: Net-(D53-Pad1) -> Net-(D53-Pad2)
- SW54 pad 1: /ROW4 -> /COL6
- SW54 pad 2: Net-(D54-Pad1) -> Net-(D54-Pad2)
- SW55 pad 1: /ROW4 -> /COL7
- SW55 pad 2: Net-(D55-Pad1) -> Net-(D55-Pad2)
- SW56 pad 1: /ROW4 -> /COL8
- SW56 pad 2: Net-(D56-Pad1) -> Net-(D56-Pad2)
- SW57 pad 1: /ROW4 -> /COL9
- SW57 pad 2: Net-(D57-Pad1) -> Net-(D57-Pad2)
- SW58 pad 1: /ROW4 -> /COL10
- SW58 pad 2: Net-(D58-Pad1) -> Net-(D58-Pad2)
- SW59 pad 1: /ROW4 -> /COL11
- SW59 pad 2: Net-(D59-Pad1) -> Net-(D59-Pad2)
- SW6 pad 1: /ROW0 -> /COL5
- SW6 pad 2: Net-(D6-Pad1) -> Net-(SW6-Pad2)
- SW7 pad 1: /ROW0 -> /COL6
- SW7 pad 2: Net-(D7-Pad1) -> Net-(D7-Pad2)
- SW8 pad 1: /ROW0 -> /COL7
- SW8 pad 2: Net-(D8-Pad1) -> Net-(SW8-Pad2)
- SW9 pad 1: /ROW0 -> /COL8
- SW9 pad 2: Net-(D9-Pad1) -> Net-(SW9-Pad2)
- U0 pad 13: /COL1 -> /ROW4
- U0 pad 14: /COL0 -> /ROW3
- U0 pad 15: /PIN15 -> /ROW2
- U0 pad 16: /ROW4 -> /ROW1
- U0 pad 17: /ROW3 -> /PIN15
- U0 pad 18: /ROW2 -> /ROW0
- U0 pad 19: /ROW1 -> /COL1
- U0 pad 20: /ROW0 -> /COL0
Routing:
- net /ROW4: track 0.00 -> 266.4 mm
- net /ROW0: track 0.00 -> 257.6 mm
- net /COL11: track 0.00 -> 249.2 mm
- net /COL10: track 0.00 -> 229.9 mm
- net /ROW1: track 0.00 -> 219.2 mm
- net /ROW2: track 0.00 -> 218.5 mm
- net /ROW3: track 0.00 -> 216.9 mm
- net /COL9: track 0.00 -> 204.4 mm
- net /COL8: track 0.00 -> 184.3 mm
- net /COL7: track 0.00 -> 164.2 mm
- net /COL6: track 0.00 -> 144.1 mm
- net /COL5: track 0.00 -> 125.6 mm
- net /COL0: track 0.00 -> 123.2 mm, vias 0 -> 1
- net /COL4: track 0.00 -> 106.9 mm
- net /COL1: track 0.00 -> 103.6 mm
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Other:
- board outline added: 230.2 x 96.8 mm
