File: kiCad/t-rex.kicad_sch (KiCad schematic)
At the start: 123 parts, among them J0 Conn_01x03, SW0 MX, SW1 MX, SW10 MX, SW11 MX, SW12 MX, SW13 MX, SW14 MX, SW15 MX, SW16 MX, SW17 MX, SW18 MX, SW19 MX, SW2 MX, SW20 MX, SW21 MX, SW22 MX, SW23 MX, SW24 MX, SW25 MX, SW26 MX, SW27 MX, SW28 MX, SW29 MX, SW3 MX, SW30 MX, SW31 MX, SW32 MX, SW33 MX, SW34 MX, SW35 MX, SW36 MX, SW37 MX, SW38 MX, SW39 MX, SW4 MX, SW40 MX, SW41 MX, SW42 MX, SW43 MX, SW44 MX, SW45 MX, SW46 MX, SW47 MX, SW48 MX, SW49 MX, SW5 MX, SW50 MX, SW51 MX, SW52 MX, SW53 MX, SW54 MX, SW55 MX, SW56 MX, SW57 MX, SW58 MX, SW59 MX, SW6 MX, SW61 MX, SW7 MX, SW8 MX, SW9 MX, U0 Sparkfun_Pro_Micro

Commit message: add traces
Connections:
- net COL0: now also U0.2 (D0/RX); no longer U0.20 (D21/A3)
- net COL1: now also U0.5 (D2); no longer U0.19 (D20/A2)
- net COL10: now also U0.19 (D20/A2); no longer U0.2 (D0/RX)
- net COL11: now also U0.20 (D21/A3); no longer U0.1 (D1/TX)
- net COL2: now also U0.6 (~D3); no longer U0.12 (~D9/A9)
- net COL3: now also U0.7 (D4/A6); no longer U0.11 (D8/A8)
- net COL4: now also U0.8 (~D5); no longer U0.10 (D7)
- net COL6: now also U0.15 (D14); no longer U0.8 (~D5)
- net COL7: now also U0.16 (D15); no longer U0.7 (D4/A6)
- net COL8: now also U0.17 (D18/A0); no longer U0.6 (~D3)
- net COL9: now also U0.18 (D19/A1); no longer U0.5 (D2)
- net PIN15: now also U0.1 (D1/TX); no longer U0.17 (D18/A0)
- net ROW0: now also U0.14 (D16); no longer U0.18 (D19/A1)
- net ROW1: now also U0.13 (~D10/A10); no longer U0.16 (D15)
- net ROW2: now also U0.10 (D7); no longer U0.15 (D14)
- net ROW3: now also U0.11 (D8/A8); no longer U0.14 (D16)
- net ROW4: now also U0.12 (~D9/A9); no longer U0.13 (~D10/A10)
Changed lines of the file:
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@@
     (stroke (width 0) (type default) (color 0 0 0 0))
   )
-  (label "COL7" (at 26.67 48.26 180)
-    (effects (font (size 1.27 1.27)) (justify right bottom))
+  (label "COL7" (at 57.15 53.34 0)
+    (effects (font (size 1.27 1.27)) (justify left bottom))
   )
   (label "COL5" (at 146.05 220.98 0)
     (effects (font (size 1.27 1.27)) (justify left bottom))
   )
-  (label "ROW3" (at 57.15 58.42 0)
-    (effects (font (size 1.27 1.27)) (justify left bottom))
+  (label "ROW3" (at 26.67 58.42 180)
+    (effects (font (size 1.27 1.27)) (justify right bottom))
   )
-  (label "COL0" (at 57.15 43.18 0)
-    (effects (font (size 1.27 1.27)) (justify left bottom))
+  (label "COL0" (at 26.67 35.56 180)
+    (effects (font (size 1.27 1.27)) (justify right bottom))
   )
-  (label "ROW0" (at 57.15 48.26 0)
+  (label "ROW0" (at 57.15 58.42 0)
     (effects (font (size 1.27 1.27)) (justify left bottom))
   )
@@
     (effects (font (size 1.27 1.27)) (justify left bottom))
   )
-  (label "ROW2" (at 57.15 55.88 0)
-    (effects (font (size 1.27 1.27)) (justify left bottom))
+  (label "ROW2" (at 26.67 55.88 180)
+    (effects (font (size 1.27 1.27)) (justify right bottom))
   )
   (label "COL5" (at 26.67 53.34 180)
     (effects (font (size 1.27 1.27)) (justify right bottom))
   )
-  (label "COL11" (at 26.67 33.02 180)
-    (effects (font (size 1.27 1.27)) (justify right bottom))
+  (label "COL11" (at 57.15 43.18 0)
+    (effects (font (size 1.27 1.27)) (justify left bottom))
   )
   (label "COL11" (at 251.46 220.98 0)
     (effects (font (size 1.27 1.27)) (justify left bottom))
   )
-  (label "COL6" (at 26.67 50.8 180)
+  (label "COL6" (at 57.15 55.88 0)
+    (effects (font (size 1.27 1.27)) (justify left bottom))
+  )
+  (label "COL3" (at 26.67 48.26 180)
     (effects (font (size 1.27 1.27)) (justify right bottom))
   )
-  (label "COL3" (at 26.67 58.42 180)
-    (effects (font (size 1.27 1.27)) (justify right bottom))
+  (label "COL9" (at 57.15 48.26 0)
+    (effects (font (size 1.27 1.27)) (justify left bottom))
   )
-  (label "COL9" (at 26.67 43.18 180)
-    (effects (font (size 1.27 1.27)) (justify right bottom))
-  )
-  (label "ROW1" (at 57.15 53.34 0)
+  (label "ROW1" (at 57.15 60.96 0)
     (effects (font (size 1.27 1.27)) (justify left bottom))
   )
@@
     (effects (font (size 1.27 1.27)) (justify left bottom))
   )
-  (label "ROW4" (at 57.15 60.96 0)
-    (effects (font (size 1.27 1.27)) (justify left bottom))
+  (label "ROW4" (at 26.67 60.96 180)
+    (effects (font (size 1.27 1.27)) (justify right bottom))
   )
-  (label "COL2" (at 26.67 60.96 180)
+  (label "COL2" (at 26.67 45.72 180)
     (effects (font (size 1.27 1.27)) (justify right bottom))
   )
@@
     (effects (font (size 1.27 1.27)) (justify left bottom))
   )
-  (label "COL10" (at 26.67 35.56 180)
-    (effects (font (size 1.27 1.27)) (justify right bottom))
+  (label "COL10" (at 57.15 45.72 0)
+    (effects (font (size 1.27 1.27)) (justify left bottom))
   )
   (label "ROW2" (at 46.99 148.59 0)
@@
     (effects (font (size 1.27 1.27)) (justify left bottom))
   )
-  (label "COL4" (at 26.67 55.88 180)
+  (label "COL4" (at 26.67 50.8 180)
     (effects (font (size 1.27 1.27)) (justify right bottom))
   )
@@
     (effects (font (size 1.27 1.27)) (justify left bottom))
   )
-  (label "COL1" (at 57.15 45.72 0)
+  (label "COL1" (at 26.67 43.18 180)
+    (effects (font (size 1.27 1.27)) (justify right bottom))
+  )
+  (label "PIN15" (at 26.67 33.02 180)
+    (effects (font (size 1.27 1.27)) (justify right bottom))
+  )
+  (label "COL8" (at 57.15 50.8 0)
     (effects (font (size 1.27 1.27)) (justify left bottom))
   )
-  (label "PIN15" (at 57.15 50.8 0)
-    (effects (font (size 1.27 1.27)) (justify left bottom))
-  )
-  (label "COL8" (at 26.67 45.72 180)
-    (effects (font (size 1.27 1.27)) (justify right bottom))
-  )
   (symbol (lib_id "Device:D_Small") (at 71.12 200.66 90) (unit 1)
