File: kiCad/t-rex.kicad_sch (KiCad schematic)
At the start: 123 parts, among them J0 Conn_01x03, SW0 MX, SW1 MX, SW10 MX, SW11 MX, SW12 MX, SW13 MX, SW14 MX, SW15 MX, SW16 MX, SW17 MX, SW18 MX, SW19 MX, SW2 MX, SW20 MX, SW21 MX, SW22 MX, SW23 MX, SW24 MX, SW25 MX, SW26 MX, SW27 MX, SW28 MX, SW29 MX, SW3 MX, SW30 MX, SW31 MX, SW32 MX, SW33 MX, SW34 MX, SW35 MX, SW36 MX, SW37 MX, SW38 MX, SW39 MX, SW4 MX, SW40 MX, SW41 MX, SW42 MX, SW43 MX, SW44 MX, SW45 MX, SW46 MX, SW47 MX, SW48 MX, SW49 MX, SW5 MX, SW50 MX, SW51 MX, SW52 MX, SW53 MX, SW54 MX, SW55 MX, SW56 MX, SW57 MX, SW58 MX, SW59 MX, SW6 MX, SW61 MX, SW7 MX, SW8 MX, SW9 MX, U0 Sparkfun_Pro_Micro

Commit message: finish routing, improve edge cuts, generate gerbers
Connections:
- net ROW0: now also U0.10 (D7); no longer U0.14 (D16)
- net ROW1: now also U0.14 (D16); no longer U0.13 (~D10/A10)
- net ROW2: now also U0.11 (D8/A8); no longer U0.10 (D7)
- net ROW3: now also U0.13 (~D10/A10); no longer U0.11 (D8/A8)
Changed lines of the file:
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@@
     (effects (font (size 1.27 1.27)) (justify left bottom))
   )
-  (label "ROW3" (at 26.67 58.42 180)
-    (effects (font (size 1.27 1.27)) (justify right bottom))
+  (label "ROW3" (at 57.15 60.96 0)
+    (effects (font (size 1.27 1.27)) (justify left bottom))
   )
   (label "COL0" (at 26.67 35.56 180)
     (effects (font (size 1.27 1.27)) (justify right bottom))
   )
-  (label "ROW0" (at 57.15 58.42 0)
-    (effects (font (size 1.27 1.27)) (justify left bottom))
+  (label "ROW0" (at 26.67 55.88 180)
+    (effects (font (size 1.27 1.27)) (justify right bottom))
   )
   (label "COL3" (at 110.49 220.98 0)
     (effects (font (size 1.27 1.27)) (justify left bottom))
   )
-  (label "ROW2" (at 26.67 55.88 180)
+  (label "ROW2" (at 26.67 58.42 180)
     (effects (font (size 1.27 1.27)) (justify right bottom))
   )
@@
     (effects (font (size 1.27 1.27)) (justify left bottom))
   )
-  (label "ROW1" (at 57.15 60.96 0)
+  (label "ROW1" (at 57.15 58.42 0)
     (effects (font (size 1.27 1.27)) (justify left bottom))
   )
