File: kiCad/t-rex.kicad_pcb (KiCad board)
At the start: 2 copper layers, 230.2 x 98 mm, 129 parts, among them J0 Conn_01x03, SW0 MX, SW1 MX, SW10 MX, SW11 MX, SW12 MX, SW13 MX, SW14 MX, SW15 MX, SW16 MX, SW17 MX, SW18 MX, SW19 MX, SW2 MX, SW20 MX, SW21 MX, SW22 MX, SW23 MX, SW24 MX, SW25 MX, SW26 MX, SW27 MX, SW28 MX, SW29 MX, SW3 MX, SW30 MX, SW31 MX, SW32 MX, SW33 MX, SW34 MX, SW35 MX, SW36 MX, SW37 MX, SW38 MX, SW39 MX, SW4 MX, SW40 MX, SW41 MX, SW42 MX, SW43 MX, SW44 MX, SW45 MX, SW46 MX, SW47 MX, SW48 MX, SW49 MX, SW5 MX, SW50 MX, SW51 MX, SW52 MX, SW53 MX, SW54 MX, SW55 MX, SW56 MX, SW57 MX, SW58 MX, SW59 MX, SW6 MX, SW61 MX, SW7 MX, SW8 MX, SW9 MX, U0 Sparkfun_Pro_Micro

Commit message: review changes
Parts:
- moved D2 0.83 mm to (75.4, 62.0)
Routing:
- net /ROW1: track 228.4 -> 231.9 mm
- net /ROW2: track 226.2 -> 228.7 mm
- net /COL0: track 123.2 -> 121.2 mm
- net +5V: track 45.5 -> 43.6 mm
- net /COL1: track 103.6 -> 102.2 mm
- net Net-(D47-Pad2): track 12.8 -> 13.8 mm
- net /ROW3: track 239.2 -> 239.8 mm

Commit message: release 1
Parts:
- added G***: LOGO, LOGO, F.Cu at (126.4, 77.5)
- added G***: LOGO, LOGO, B.Cu at (171.1, 77.5)
- moved D23 0.75 mm to (247.7, 61.8)
Routing:
- net /COL11: track 249.2 -> 253.1 mm
- net /COL10: track 229.6 -> 232.2 mm
- net /COL9: track 204.4 -> 206.6 mm
- net GND: track 88.7 -> 87.2 mm
- net /COL8: track 184.3 -> 185.5 mm
- net /ROW1: track 231.9 -> 231.3 mm

Commit message: align silkscreen
Parts:
- moved ? 19.1 mm to (147.6, 42.9)
- moved G*** 3.47 mm to (123.8, 75.1)
- moved G*** 2.32 mm to (171.4, 75.2)
Changed lines of the file:
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@@
   )
   (footprint "LOGO" (layer "F.Cu")
-    (at 126.365 77.47)
+    (at 123.828998 75.100522)
     (attr board_only exclude_from_pos_files exclude_from_bom)
     (fp_text reference "G***" (at 0 0) (layer "F.SilkS")
@@
   )
   (footprint "" (layer "F.Cu")
-    (at 147.6375 61.9125)
+    (at 147.6375 42.8625)
     (fp_text reference "" (at 0 0) (layer "F.SilkS")
       (effects (font (size 1.27 1.27) (thickness 0.15)))
@@
   )
   (footprint "LOGO" (layer "B.Cu")
-    (at 171.065003 77.513522 180)
+    (at 171.446003 75.227522 180)
     (attr board_only exclude_from_pos_files exclude_from_bom)
     (fp_text reference "G***" (at 0 0) (layer "B.SilkS")

Commit message: new layout with numbpad
Parts:
- removed G*** (x2): LOGO, LOGO
- U0: moved to F.Cu
- moved SW61 207.9 mm to (233.0, 164.9), turned to 78 degrees
- moved D0 199.7 mm to (188.7, 182.4)
- moved D1 199.7 mm to (193.5, 188.7)
- moved SW0 199.7 mm to (179.2, 179.2)
- moved SW1 199.7 mm to (198.3, 179.2)
- moved SW2 199.7 mm to (217.3, 179.2)
- moved J0 149.9 mm to (181.5, 107.3)
- moved D5 149.4 mm to (226.8, 163.0)
- moved D3 149.4 mm to (188.7, 163.0)
- moved D4 149.4 mm to (207.8, 163.0)
- moved SW3 149.4 mm to (179.2, 160.0)
- moved SW4 149.4 mm to (198.3, 160.0)
- moved SW5 149.4 mm to (217.3, 160.0)
- moved U0 130.0 mm to (198.7, 95.2)
- moved D6 109.8 mm to (188.9, 143.9)
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Routing:
- net /ROW0: track 257.9 -> 0.00 mm
- net /COL11: track 253.1 -> 0.00 mm
- net /COL10: track 232.2 -> 0.00 mm
- net /COL9: track 206.6 -> 0.00 mm
- net /COL8: track 185.5 -> 0.00 mm
- net /COL7: track 164.2 -> 0.00 mm
- net /ROW3: track 239.8 -> 95.3 mm
- net /COL6: track 144.1 -> 0.00 mm
- net /ROW1: track 231.3 -> 95.3 mm
- net /ROW2: track 228.7 -> 95.3 mm
- net /COL5: track 125.8 -> 0.00 mm
- net /COL4: track 107.4 -> 0.00 mm
- net GND: track 87.2 -> 0.00 mm
- net /COL3: track 86.4 -> 0.00 mm
- net /ROW4: track 266.3 -> 186.3 mm
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Other:
- board outline removed

Commit message: add traces
Parts:
- removed ? (x6): , 
- moved D2 155.2 mm to (226.8, 185.0), turned to 90 degrees
- moved SW61 119.0 mm to (219.9, 46.6), turned to -102 degrees
- moved J0 96.2 mm to (254.1, 44.0)
- moved D1 15.6 mm to (207.8, 182.4), turned to 90 degrees
- moved D11 15.4 mm to (226.8, 125.5), turned to 90 degrees
- moved D17 1.08 mm to (170.5, 107.8)
- moved D9 0.54 mm to (188.7, 125.2)
- moved D10 0.38 mm to (207.5, 125.0)
- moved U0 0.20 mm to (198.5, 95.2)
Connections:
- U0 pad 1: /COL11 -> /PIN15
- U0 pad 10: /COL4 -> /ROW2
- U0 pad 11: /COL3 -> /ROW3
- U0 pad 12: /COL2 -> /ROW4
- U0 pad 13: /ROW4 -> /ROW1
- U0 pad 14: /ROW3 -> /ROW0
- U0 pad 15: /ROW2 -> /COL6
- U0 pad 16: /ROW1 -> /COL7
- U0 pad 17: /PIN15 -> /COL8
- U0 pad 18: /ROW0 -> /COL9
- U0 pad 19: /COL1 -> /COL10
- U0 pad 2: /COL10 -> /COL0
- U0 pad 20: /COL0 -> /COL11
- U0 pad 5: /COL9 -> /COL1
- U0 pad 6: /COL8 -> /COL2
- U0 pad 7: /COL7 -> /COL3
- U0 pad 8: /COL6 -> /COL4
Routing:
- net /COL11: track 0.00 -> 478.0 mm
- net /COL10: track 0.00 -> 417.6 mm
- net /COL9: track 0.00 -> 351.0 mm
- net /COL8: track 0.00 -> 257.0 mm
- net /COL7: track 0.00 -> 238.2 mm
- net /COL3: track 0.00 -> 225.5 mm
- net /COL6: track 0.00 -> 217.1 mm
- net /COL4: track 0.00 -> 213.0 mm
- net /COL2: track 93.3 -> 293.0 mm
- net /COL1: track 114.0 -> 313.5 mm
- net /ROW0: track 0.00 -> 194.8 mm
- net /COL5: track 0.00 -> 194.2 mm
- net /COL0: track 199.8 -> 337.4 mm, vias 1 -> 0
- net /ROW2: track 95.3 -> 189.8 mm
- net /ROW3: track 95.3 -> 176.8 mm
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Other:
- board outline added: 307.8 x 120.6 mm

Commit message: finish routing, improve edge cuts, generate gerbers
Parts:
- added ?: , , F.Cu at (328.2, 129.5)
- added ?: , , F.Cu at (198.4, 103.8)
- added ?: , LOGO, F.Cu at (231.1, 183.1)
- added ?: , , F.Cu at (320.3, 92.2)
- added ?: , , F.Cu at (68.3, 129.6)
- added ?: , , F.Cu at (76.2, 92.4)
- added ?: , , F.Cu at (198.3, 169.5)
- added ?: , LOGO, F.Cu at (165.4, 183.2)
- added G***: LOGO, LOGO, B.Cu at (257.4, 128.2)
- added G***: LOGO, LOGO, B.Cu at (139.2, 128.3)
- moved J0 66.6 mm to (200.9, 84.2)
- moved SW61 53.6 mm to (198.2, 95.6), turned to 0 degrees
- moved D29 32.8 mm to (140.2, 105.9), turned to -12 degrees
- moved D53 19.8 mm to (147.3, 146.2), turned to -12 degrees
- moved D41 19.7 mm to (151.3, 127.9), turned to -12 degrees
- moved D17 15.2 mm to (155.3, 109.0), turned to -12 degrees
- moved D2 1.35 mm to (225.4, 185.1)
- moved D11 1.20 mm to (225.7, 125.4)
- moved D8 1.12 mm to (225.8, 143.9)
- moved D5 1.05 mm to (225.8, 163.0)
- moved SW6 0.13 mm to (179.2, 140.8)
- moved SW8 0.13 mm to (217.3, 140.8)
Connections:
- U0 pad 10: /ROW2 -> /ROW0
- U0 pad 11: /ROW3 -> /ROW2
- U0 pad 13: /ROW1 -> /ROW3
- U0 pad 14: /ROW0 -> /ROW1
Routing:
- net /ROW4: track 186.3 -> 339.8 mm
- net /ROW3: track 176.8 -> 300.9 mm
- net /ROW2: track 189.8 -> 295.5 mm
- net /ROW1: track 173.3 -> 264.4 mm
- net /ROW0: track 194.8 -> 239.1 mm, vias 0 -> 1
- net Net-(SW61-Pad1): track 0.00 -> 13.4 mm
- net +5V: track 0.00 -> 12.2 mm
- net /PIN15: track 0.00 -> 12.2 mm
- net Net-(D29-Pad2): track 7.12 -> 17.2 mm
- net GND: track 18.8 -> 27.7 mm
- net Net-(D54-Pad2): track 0.58 -> 7.92 mm
- net Net-(D57-Pad2): track 0.00 -> 7.18 mm
- net Net-(D56-Pad2): track 0.00 -> 7.18 mm
- net Net-(D55-Pad2): track 0.00 -> 7.18 mm
- net Net-(D6-Pad2): track 0.00 -> 7.18 mm
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Other:
- board size 307.8 x 120.6 mm -> 309.9 x 120.6 mm
- board text added: "@SylivanKenobi"
