File: kiCad/t-rex.kicad_pcb (KiCad board)
At the start: 2 copper layers, 230.2 x 98 mm, 131 parts, among them J0 Conn_01x03, SW0 MX, SW1 MX, SW10 MX, SW11 MX, SW12 MX, SW13 MX, SW14 MX, SW15 MX, SW16 MX, SW17 MX, SW18 MX, SW19 MX, SW2 MX, SW20 MX, SW21 MX, SW22 MX, SW23 MX, SW24 MX, SW25 MX, SW26 MX, SW27 MX, SW28 MX, SW29 MX, SW3 MX, SW30 MX, SW31 MX, SW32 MX, SW33 MX, SW34 MX, SW35 MX, SW36 MX, SW37 MX, SW38 MX, SW39 MX, SW4 MX, SW40 MX, SW41 MX, SW42 MX, SW43 MX, SW44 MX, SW45 MX, SW46 MX, SW47 MX, SW48 MX, SW49 MX, SW5 MX, SW50 MX, SW51 MX, SW52 MX, SW53 MX, SW54 MX, SW55 MX, SW56 MX, SW57 MX, SW58 MX, SW59 MX, SW6 MX, SW61 MX, SW7 MX, SW8 MX, SW9 MX, U0 Sparkfun_Pro_Micro

Commit message: update to kicad 7, cleanup repo
Parts:
- removed ? (x6): , 

Commit message: fix missing mount holes in pcb
Parts:
- added ?: , , F.Cu at (148.0, 100.1)
- added ?: , , F.Cu at (52.4, 42.9)
- added ?: , , F.Cu at (147.5, 61.8)
- added ?: , , F.Cu at (243.1, 43.0)
- added ?: , , F.Cu at (52.2, 100.1)
- added ?: , , F.Cu at (243.1, 99.8)
Changed lines of the file:
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@@
     )
   )
+  (footprint "" (layer "F.Cu")
+    (at 148 100.075)
+    (fp_text reference "" (at 0 0) (layer "F.SilkS")
+        (effects (font (size 1.27 1.27) (thickness 0.15)))
+    )
+    (fp_text value "" (at 0 0) (layer "F.SilkS")
+        (effects (font (size 1.27 1.27) (thickness 0.15)))
+    )
+    (pad "1" thru_hole circle (at -0.513086 -0.064351) (size 4.4 4.4) (drill 2.2) (layers "*.Cu" "*.Mask"))
+  )
   (footprint "Diode_THT:D_DO-35_SOD27_P7.62mm_Horizontal" (layer "F.Cu")
     (at 147.6375 36.35375 90)
@@
     )
   )
+  (footprint "" (layer "F.Cu")
+    (at 52.4 42.85)
+    (fp_text reference "" (at 0 0) (layer "F.SilkS")
+        (effects (font (size 1.27 1.27) (thickness 0.15)))
+    )
+    (fp_text value "" (at 0 0) (layer "F.SilkS")
+        (effects (font (size 1.27 1.27) (thickness 0.15)))
+    )
+    (pad "1" thru_hole circle (at -0.0125 0.0125) (size 4.4 4.4) (drill 2.2) (layers "*.Cu" "*.Mask"))
+  )
   (footprint "MX_Alps_Hybrid:MX-1U-NoLED" (layer "F.Cu")
     (at 138.1125 33.3375)
@@
       (net 49 "Net-(D28-A)") (pinfunction "2") (pintype "passive"))
   )
+  (footprint "" (layer "F.Cu")
+    (at 147.5 61.825)
+    (fp_text reference "" (at 0 0) (layer "F.SilkS")
+        (effects (font (size 1.27 1.27) (thickness 0.15)))
+    )
+    (fp_text value "" (at 0 0) (layer "F.SilkS")
+        (effects (font (size 1.27 1.27) (thickness 0.15)))
+    )
+    (pad "1" thru_hole circle (at 0.1375 0.0875) (size 4.4 4.4) (drill 2.2) (layers "*.Cu" "*.Mask"))
+  )
   (footprint "MX_Alps_Hybrid:MX-1U-NoLED" (layer "F.Cu")
     (at 61.9125 52.3875)
@@
       (net 69 "Net-(D48-A)") (pinfunction "2") (pintype "passive"))
   )
+  (footprint "" (layer "F.Cu")
+    (at 243.05 43)
+    (fp_text reference "" (at 0 0) (layer "F.SilkS")
+        (effects (font (size 1.27 1.27) (thickness 0.15)))
+    )
+    (fp_text value "" (at 0 0) (layer "F.SilkS")
+        (effects (font (size 1.27 1.27) (thickness 0.15)))
+    )
+    (pad "1" thru_hole circle (at -0.1625 -0.1375) (size 4.4 4.4) (drill 2.2) (layers "*.Cu" "*.Mask"))
+  )
   (footprint "MX_Alps_Hybrid:MX-1U-NoLED" (layer "F.Cu")
     (at 138.1125 71.4375)
@@
     )
   )
+  (footprint "" (layer "F.Cu")
+    (at 52.225 100.075)
+    (fp_text reference "" (at 0 0) (layer "F.SilkS")
+        (effects (font (size 1.27 1.27) (thickness 0.15)))
+    )
+    (fp_text value "" (at 0 0) (layer "F.SilkS")
+        (effects (font (size 1.27 1.27) (thickness 0.15)))
+    )
+    (pad "1" thru_hole circle (at 0.1625 -0.0625) (size 4.4 4.4) (drill 2.2) (layers "*.Cu" "*.Mask"))
+  )
   (footprint "Diode_THT:D_DO-35_SOD27_P7.62mm_Horizontal" (layer "F.Cu")
     (at 204.7875 113.3475 90)
@@
       (net 52 "Net-(D31-A)") (pinfunction "2") (pintype "passive"))
   )
+  (footprint "" (layer "F.Cu")
+    (at 243.05 99.825)
+    (fp_text reference "" (at 0 0) (layer "F.SilkS")
+        (effects (font (size 1.27 1.27) (thickness 0.15)))
+    )
+    (fp_text value "" (at 0 0) (layer "F.SilkS")
+        (effects (font (size 1.27 1.27) (thickness 0.15)))
+    )
+    (pad "1" thru_hole circle (at -0.1625 0.1875) (size 4.4 4.4) (drill 2.2) (layers "*.Cu" "*.Mask"))
+  )
   (footprint "LOGO" (layer "B.Cu")
